Commit message: add offboard node and camera transfer stuff, decrease the sample num of lidar in order to accelerate the sim time add px4 sim in the gazebo, the sim time factor is 0.1 when processing

File: src/wheeltec_robot_gazebo/wheeltec_description/urdf/livox_mid360.xacro (robot description, xacro)
@@ -8,5 +8,5 @@
     <xacro:property name="laser_min_range" value="0.1"/>
     <xacro:property name="laser_max_range" value="40"/>
-    <xacro:property name="samples" value="20000"/>
+    <xacro:property name="samples" value="10000"/>
     <xacro:property name="downsample" value="1"/>
     <xacro:macro name="laser_livox" params="NS">
@@ -44,5 +44,5 @@
                         <scan>
                             <horizontal>
-                                <samples>100</samples>
+                                <samples>50</samples>
                                 <resolution>1</resolution>
                                 <min_angle>-${M_PI}</min_angle>
@@ -50,5 +50,5 @@
                             </horizontal>
                             <vertical>
-                                <samples>100</samples>
+                                <samples>50</samples>
                                 <resolution>1</resolution>
                                 <min_angle>${-M_PI}</min_angle>

Commit message: offboard setting success

File: src/wheeltec_robot_gazebo/wheeltec_description/urdf/livox_mid360.xacro (robot description, xacro)
@@ -2,5 +2,5 @@
 <robot name="wheeltec"
     xmlns:xacro="http://www.ros.org/wiki/xacro">
-    <xacro:property name="update_rate" value="30"/>
+    <xacro:property name="update_rate" value="10"/>
     <xacro:property name="resolution" value="0.01"/>
     <xacro:property name="noise_mean" value="0.01"/>

Commit message: add offboard and camera ns, uav still got tf problem

File: src/wheeltec_robot_gazebo/wheeltec_description/urdf/livox_mid360.xacro (robot description, xacro)
@@ -2,5 +2,5 @@
 <robot name="wheeltec"
     xmlns:xacro="http://www.ros.org/wiki/xacro">
-    <xacro:property name="update_rate" value="10"/>
+    <xacro:property name="update_rate" value="20"/>
     <xacro:property name="resolution" value="0.01"/>
     <xacro:property name="noise_mean" value="0.01"/>
